Commit message: functionnal gazebo simulation

File: simulation/urdf/quadrus.urdf (robot description, URDF)
Before this commit: robot quadrus, 9 links, 8 joints
Links:
- added link back_left_dummy
- added link back_right_dummy
- added link front_left_dummy
- added link front_right_dummy
- link base_link: geometry visual box size=0.05 0.05 0.05; visual box size=0.05 0.05 0.05
Joints:
- added joint joint_back_left_hip: type continuous, parent base_link, child back_left_dummy, origin xyz=-0.08 0.075 0 rpy=0 0 0, axis 1 0 0
- added joint joint_back_right_hip: type continuous, parent base_link, child back_right_dummy, origin xyz=-0.08 -0.075 0 rpy=0 0 0, axis 1 0 0
- added joint joint_front_left_hip: type continuous, parent base_link, child front_left_dummy, origin xyz=0.08 0.075 0 rpy=0 0 0, axis 1 0 0
- added joint joint_front_right_hip: type continuous, parent base_link, child front_right_dummy, origin xyz=0.08 -0.075 0 rpy=0 0 0, axis 1 0 0
- joint joint_back_left_lowerleg: axis 1 0 0 -> 0 1 0; origin xyz=0.10 0 0 rpy=0 -1.55 0 -> xyz=-0.10 0 0 rpy=0 1.5708 0
- joint joint_back_left_upperleg: axis 1 0 0 -> 0 1 0; origin xyz=-0.08 -0.075 0 rpy=0 2.5 0 -> xyz=-0.05 0 0 rpy=0 -0.7854 0; parent base_link -> back_left_dummy
- joint joint_back_right_lowerleg: axis 1 0 0 -> 0 1 0; origin xyz=0.10 0 0 rpy=0 -1.55 0 -> xyz=-0.10 0 0 rpy=0 1.5708 0
- joint joint_back_right_upperleg: axis 1 0 0 -> 0 1 0; origin xyz=-0.08 0.075 0 rpy=0 2.5 0 -> xyz=-0.05 0 0 rpy=0 -0.7854 0; parent base_link -> back_right_dummy
- joint joint_front_left_lowerleg: axis 1 0 0 -> 0 1 0; origin xyz=0.10 0 0 rpy=0 -1.55 0 -> xyz=-0.10 0 0 rpy=0 1.5708 0
- joint joint_front_left_upperleg: axis 1 0 0 -> 0 1 0; origin xyz=0.08 -0.075 0 rpy=0 2.5 0 -> xyz=-0.05 0 0 rpy=0 -0.7854 0; parent base_link -> front_left_dummy
- joint joint_front_right_lowerleg: axis 1 0 0 -> 0 1 0; origin xyz=0.10 0 0 rpy=0 -1.55 0 -> xyz=-0.10 0 0 rpy=0 1.5708 0
- joint joint_front_right_upperleg: axis 1 0 0 -> 0 1 0; origin xyz=0.08 0.075 0 rpy=0 2.5 0 -> xyz=-0.05 0 0 rpy=0 -0.7854 0; parent base_link -> front_right_dummy
