Commit message: urdf test files

File: ros_packages/qd_simulation/robot_description/quadrus_forced.xacro (robot description, xacro)
@@ -14,10 +14,4 @@
 	<xacro:include filename="$(find qd_simulation)/robot_description/quadrus.gazebo" />
 	<!-- Used for fixing robot to Gazebo 'base_link' -->
-	<link name="world"/>
-	<joint name="fixed" type="fixed">
-		<parent link="world"/>
-		<child link="base_link"/>
-		<origin xyz="0 0 1"/>
-	</joint>
 	<link name="base_link">
 		<visual>
@@ -35,13 +29,7 @@
 			<material name="blue"/>
 		</visual>
-		<collision>
-			<origin xyz="0 0 0" rpy="0 0 0" />
-			<geometry>
-				<box size="0.4172 0.116 0.03035"/>
-			</geometry>
-		</collision>
 		<inertial>
 			<mass value="0.800"/>
-			<inertia ixx="0.00228" ixy="0.0" ixz="0.0" iyy="0.01125" iyz="0.0" izz="0.01326"/>
+			<inertia ixx="0.1" ixy="0.1" ixz="0.10" iyy="0.1" iyz="0.1" izz="0.1"/>
 		</inertial>
 	</link>
@@ -57,14 +45,8 @@
 					<material name="red"/>
 				</visual>
-				<collision>
-					<origin xyz="0 0 0" rpy="0 0 0" />
-					<geometry>
-						<box size="0.060 0.035 0.078"/>
-					</geometry>
-				</collision>
 				<inertial>
 					<mass value="0.37017"/>
 					<origin xyz="0.00025 0.0063 0.04447"/>
-					<inertia ixx="0.00114" ixy="0.0" ixz="-0.00004" iyy="0.00074" iyz="-0.00021" izz="0.00064"/>
+					<inertia ixx="0.1" ixy="0.1" ixz="0.1" iyy="0.1" iyz="0.1" izz="0.1"/>
 				</inertial>
 			</link>
@@ -109,14 +91,8 @@
 					<material name="blue"/>
 				</visual>
-				<collision>
-					<origin xyz="-0.07 0 0" rpy="0 0 0" />
-					<geometry>
-						<box size="${upperleg_length+0.03}  0.0365 0.026"/>
-					</geometry>
-				</collision>
 				<inertial>
 					<mass value="0.35314"/>
 					<origin xyz="-0.06146 -0.00199 0.00083"/>
-					<inertia ixx="0.00015" ixy="-0.00003" ixz="0.00004" iyy="0.00074" iyz="0.0" izz="0.00083"/>
+					<inertia ixx="0.1" ixy="0.1" ixz="0.1" iyy="0.1" iyz="0.1" izz="0.1"/>
 				</inertial>
 			</link>
@@ -155,14 +131,8 @@
 					<material name="blue"/>
 				</visual>
-				<collision>
-					<origin xyz="0.075 0 0" rpy="0 0 0" />
-					<geometry>
-						<box size="${lowerleg_length+0.03} 0.02 0.03"/>
-					</geometry>
-				</collision>
 				<inertial>
 					<origin xyz=" 0.05439 0.00478 0"/>
 					<mass value="0.23649"/>
-					<inertia ixx="0.0" ixy="0.0" ixz="0.0" iyy="0.00052" iyz="0.0" izz="0.00054"/>
+					<inertia ixx="0.1" ixy="0.1" ixz="0.1" iyy="0.1" iyz="0.1" izz="0.1"/>
 				</inertial>
 			</link>
@@ -195,13 +165,7 @@
 					<material name="green"/>
 				</visual>
-				<collision>
-					<origin xyz="0 0 0" rpy="0 0 0" />
-					<geometry>
-						<sphere radius = "0.02"/>
-					</geometry>
-				</collision>
 				<inertial>
 					<mass value="0.02"/>
-					<inertia ixx="0.0" ixy="0.0" ixz="0.0" iyy="0.0" iyz="0.0" izz="0.0"/>
+					<inertia ixx="0.1" ixy="0.1" ixz="0.1" iyy="0.1" iyz="0.1" izz="0.1"/>
 				</inertial>
 			</link>

File: ros_packages/qd_simulation/robot_description/quadrus_nonzero.xacro (robot description, xacro)
@@ -14,10 +14,4 @@
 	<xacro:include filename="$(find qd_simulation)/robot_description/quadrus.gazebo" />
 	<!-- Used for fixing robot to Gazebo 'base_link' -->
-	<link name="world"/>
-	<joint name="fixed" type="fixed">
-		<parent link="world"/>
-		<child link="base_link"/>
-		<origin xyz="0 0 1"/>
-	</joint>
 	<link name="base_link">
 		<visual>
@@ -66,5 +60,5 @@
 					<mass value="0.37017"/>
 					<origin xyz="0.00025 0.0063 0.04447"/>
-					<inertia ixx="0.00114" ixy="0.0" ixz="-0.00004" iyy="0.00074" iyz="-0.00021" izz="0.00064"/>
+					<inertia ixx="0.00114" ixy="0.0" ixz="0.0" iyy="0.0" iyz="0.0" izz="0.0"/>
 				</inertial>
 			</link>
@@ -118,5 +112,5 @@
 					<mass value="0.35314"/>
 					<origin xyz="-0.06146 -0.00199 0.00083"/>
-					<inertia ixx="0.00015" ixy="-0.00003" ixz="0.00004" iyy="0.00074" iyz="0.0" izz="0.00083"/>
+					<inertia ixx="0.0" ixy="0.0" ixz="0.0" iyy="0.0" iyz="0.0" izz="0.0"/>
 				</inertial>
 			</link>
@@ -164,5 +158,5 @@
 					<origin xyz=" 0.05439 0.00478 0"/>
 					<mass value="0.23649"/>
-					<inertia ixx="0.0" ixy="0.0" ixz="0.0" iyy="0.00052" iyz="0.0" izz="0.00054"/>
+					<inertia ixx="0.0" ixy="0.0" ixz="0.0" iyy="0.0" iyz="0.0" izz="0.0"/>
 				</inertial>
 			</link>
