Commit message: benchmark controller tuning

File: ros_packages/qd_simulation/robot_description/motor_benchmark.xacro (robot description, xacro)
@@ -3,5 +3,5 @@
 	<!-- Import Rviz colors -->
 	<xacro:include filename="$(find qd_simulation)/robot_description/materials.xacro" />
-	<!-- Import all Gazebo-customization elements, including Gazebo colors -->
+    <!-- Import all Gazebo-customization elements, including Gazebo colors -->
 	<xacro:include filename="$(find qd_simulation)/robot_description/quadrus.gazebo" />
 	<!-- Used for fixing robot to Gazebo 'base_link' -->
@@ -15,4 +15,9 @@
 			<material name="blue" />
 		</visual>
+        <inertial>
+            <origin xyz="0 0 0"/>
+            <mass value="0.15"/>
+            <inertia ixx="0.0" ixy="0.0" ixz="0.0" iyy="0.0" iyz="0.0" izz="0.0"/>
+        </inertial>
 	</link>
     <link name="baton">
@@ -53,5 +58,5 @@
         <child link="baton"/>
         <origin xyz="0 0.06 0.45" rpy="-1.570 1.57 0" />
-        <axis xyz="0 1 0" />
+        <axis xyz="0 0 1" />
     </joint>
     <joint name="fixed2" type="fixed">
@@ -63,5 +68,5 @@
     <transmission name="transmission_J1">
         <type>transmission_interface/SimpleTransmission</type>
-        <joint name="$J1">
+        <joint name="J1">
             <hardwareInterface>hardware_interface/EffortJointInterface</hardwareInterface>
         </joint>

Commit message: Modified urdf collision volumes

File: ros_packages/qd_simulation/robot_description/motor_benchmark.xacro (robot description, xacro)
@@ -30,7 +30,7 @@
         </visual>
         <inertial>
-            <origin xyz="0 0 0"/>
-            <mass value="0.15"/>
-            <inertia ixx="0.0" ixy="0.0" ixz="0.0" iyy="0.0" iyz="0.0" izz="0.0"/>
+            <origin xyz="0.0875 0 0"/>
+            <mass value="0.015"/>
+            <inertia ixx="0.0" ixy="0.0" ixz="0.0" iyy="0.0" iyz="0.0" izz="0.000039062"/>
         </inertial>
     </link>
@@ -46,5 +46,5 @@
             <origin xyz="0 0 0"/>
             <mass value="0.163"/>
-            <inertia ixx="0.0" ixy="0.0" ixz="0.0" iyy="0.0" iyz="0.0" izz="0.0"/>
+            <inertia ixx="0.0" ixy="0.0" ixz="0.0" iyy="0.0" iyz="0.0" izz="0.000050625"/>
         </inertial>
     </link>

File: ros_packages/qd_simulation/robot_description/quadrus.xacro (robot description, xacro)
@@ -32,5 +32,6 @@
 			<origin xyz="0 0 0" rpy="0 0 0" />
 			<geometry>
-				<mesh filename="package://qd_simulation/robot_description/mesh/body.dae"/>
+				<box size="0.417 0.116 0.03"/>
+				<!-- mesh filename="package://qd_simulation/robot_description/mesh/body.dae"/-->
 			</geometry>
 		</collision>
@@ -61,13 +62,15 @@
 				<collision>
 					<xacro:if value="${lat == 'left'}">
-						<origin xyz="0 0 0" rpy="0 0 0" />
-						<geometry>
-							<mesh filename="package://qd_simulation/robot_description/mesh/left_hip.dae"/>
-						</geometry>
-					</xacro:if>
-					<xacro:if value="${lat == 'right'}">
-						<origin xyz="0 0 0" rpy="0 0 0" />
-						<geometry>
-							<mesh filename="package://qd_simulation/robot_description/mesh/right_hip.dae"/>
+						<origin xyz="0.014 0.04125 0.0147" rpy="0 0 0" />
+						<geometry>
+							<box size="0.064 0.103 0.0685"/>
+							<!-- mesh filename="package://qd_simulation/robot_description/mesh/left_hip.dae"/-->
+						</geometry>
+					</xacro:if>
+					<xacro:if value="${lat == 'right'}">
+						<origin xyz="0.014 -0.04125 0.0147" rpy="0 0 0" />
+						<geometry>
+							<box size="0.064 0.103 0.0685"/>
+							<!-- mesh filename="package://qd_simulation/robot_description/mesh/right_hip.dae"/-->
 						</geometry>
 					</xacro:if>
@@ -108,5 +111,5 @@
 			<gazebo reference="link_${long}_${lat}_hip">
 				<material>Gazebo/Red</material>
-				<selfCollide>true</selfCollide>
+				<!-- selfCollide>true</selfCollide -->
 				<gravity>true</gravity>
 			</gazebo>
@@ -131,13 +134,15 @@
 				<collision>
 					<xacro:if value="${lat == 'left'}">
-						<origin xyz="0 0 0" rpy="0 0 0" />
-						<geometry>
-							<mesh filename="package://qd_simulation/robot_description/mesh/left_femur.dae"/>
-						</geometry>
-					</xacro:if>
-					<xacro:if value="${lat == 'right'}">
-						<origin xyz="0 0 0" rpy="0 0 0" />
-						<geometry>
-							<mesh filename="package://qd_simulation/robot_description/mesh/right_femur.dae"/>
+						<origin xyz="-0.066 0 -0.008" rpy="0 0 0" />
+						<geometry>
+							<box size="0.172 0.073 0.046"/>
+							<!-- mesh filename="package://qd_simulation/robot_description/mesh/left_femur.dae"/-->
+						</geometry>
+					</xacro:if>
+					<xacro:if value="${lat == 'right'}">
+						<origin xyz="-0.066 0 -0.008" rpy="0 0 0" />
+						<geometry>
+							<box size="0.172 0.073 0.046"/>
+							<!-- mesh filename="package://qd_simulation/robot_description/mesh/right_femur.dae"/-->
 						</geometry>
 					</xacro:if>
@@ -172,5 +177,5 @@
 			<gazebo reference="link_${long}_${lat}_upperleg">
 				<material>Gazebo/White</material>
-				<selfCollide>true</selfCollide>
+				<!-- selfCollide>true</selfCollide -->
 				<gravity>true</gravity>
 			</gazebo>
@@ -195,13 +200,15 @@
 				<collision>
 					<xacro:if value="${lat == 'left'}">
-						<origin xyz="0 0 0" rpy="0 0 0" />
-						<geometry>
-							<mesh filename="package://qd_simulation/robot_description/mesh/left_tibia.dae"/>
-						</geometry>
-					</xacro:if>
-					<xacro:if value="${lat == 'right'}">
-						<origin xyz="0 0 0" rpy="0 0 0" />
-						<geometry>
-							<mesh filename="package://qd_simulation/robot_description/mesh/right_tibia.dae"/>
+						<origin xyz="0.055 0 0" rpy="0 0 0" />
+						<geometry>
+							<box size="0.15 0.048 0.028"/>
+							<!-- mesh filename="package://qd_simulation/robot_description/mesh/left_tibia.dae"/-->
+						</geometry>
+					</xacro:if>
+					<xacro:if value="${lat == 'right'}">
+						<origin xyz="0.055 0 0" rpy="0 0 0" />
+						<geometry>
+							<box size="0.15 0.048 0.028"/>
+							<!-- mesh filename="package://qd_simulation/robot_description/mesh/right_tibia.dae"/-->
 						</geometry>
 					</xacro:if>
@@ -231,5 +238,5 @@
 			<gazebo reference="link_${long}_${lat}_lowerleg">
 				<material>Gazebo/White</material>
-				<selfCollide>true</selfCollide>
+				<!-- selfCollide>true</selfCollide -->
 				<gravity>true</gravity>
 			</gazebo>
@@ -246,10 +253,11 @@
 					<origin xyz="0 0 0" rpy="0 0 0" />
 					<geometry>
-						<mesh filename="package://qd_simulation/robot_description/mesh/tpe_tip.dae"/>
+						<sphere radius = "0.02"/>
+						<!-- mesh filename="package://qd_simulation/robot_description/mesh/tpe_tip.dae"/-->
 					</geometry>
 				</collision>
 				<inertial>
 					<mass value="0.003"/>
-					<inertia ixx="0.0" ixy="0.0" ixz="0.0" iyy="0.0" iyz="0.0" izz="0.0"/>
+					<inertia ixx="0.00001" ixy="0.0" ixz="0.0" iyy="0.00001" iyz="0.0" izz="0.00001"/>
 				</inertial>
 			</link>
@@ -261,4 +269,6 @@
 			<gazebo reference="link_${long}_${lat}_paw">
 				<material>Gazebo/Green</material>
+				<!-- selfCollide>true</selfCollide -->
+				<gravity>true</gravity>
 			</gazebo>
 	</xacro:macro>
@@ -267,4 +277,3 @@
 	<xacro:quadrus_leg long="back" lat="left" id="3"/>
 	<xacro:quadrus_leg long="back" lat="right" id="4"/>
-	<selfCollide>true</selfCollide>
 </robot>
