Commit message: rosserial integration

File: ros_packages/qd_simulation/robot_description/quadrus.xacro (robot description, xacro)
@@ -123,8 +123,8 @@
 				<child link="link_${long}_${lat}_upperleg"/>
 				<xacro:if value="${lat == 'left'}">
-					<origin xyz="0 ${hip_offset} 0" rpy="0 -0.7854 0" />
+					<origin xyz="0 ${hip_offset} 0" rpy="0 0 0" />
 				</xacro:if>
 				<xacro:if value="${lat == 'right'}">
-					<origin xyz="0 ${-hip_offset} 0" rpy="0 -0.7854 0" />
+					<origin xyz="0 ${-hip_offset} 0" rpy="0 0 0" />
 				</xacro:if>
 				<axis xyz="0 1 0" />

Commit message: Updated urdf file

File: ros_packages/qd_simulation/robot_description/quadrus.xacro (robot description, xacro)
@@ -3,10 +3,10 @@
 	<!-- Constants for robot dimensions, mass and inertia-->
 	<xacro:property name="PI" value="3.1415926535897931"/>
-	<xacro:property name="hip_offset" value="0.04" />
-	<xacro:property name="upperleg_length" value="0.150" />
-	<xacro:property name="lowerleg_length" value="0.150" />
-	<xacro:property name="rear_hip_long_offset" value="-0.12" />
-	<xacro:property name="hip_long_center_dist" value="0.24" />
-	<xacro:property name="hip_lat_center_dist" value="0.15" />
+	<xacro:property name="hip_offset" value="0.05755" />
+	<xacro:property name="upperleg_length" value="0.140" />
+	<xacro:property name="lowerleg_length" value="0.14833" />
+	<xacro:property name="rear_hip_long_offset" value="-0.148" />
+	<xacro:property name="hip_long_center_dist" value="0.268" />
+	<xacro:property name="hip_lat_center_dist" value="0.158" />
 	<!-- Import Rviz colors -->
 	<xacro:include filename="$(find qd_simulation)/robot_description/materials.xacro" />
@@ -24,5 +24,5 @@
 			<origin xyz="0 0 0" rpy="0 0 0" />
 			<geometry>
-				<box size="0.30 0.10 0.07"/>
+				<box size="0.4172 0.116 0.03035"/>
 			</geometry>
 			<material name="blue" />
@@ -31,5 +31,5 @@
 			<origin xyz="0 0 0" rpy="0 0 0" />
 			<geometry>
-				<box size="0.2 0.18 0.07"/>
+				<box size="0.2 0.2 0.03035"/>
 			</geometry>
 			<material name="blue"/>
@@ -38,10 +38,10 @@
 			<origin xyz="0 0 0" rpy="0 0 0" />
 			<geometry>
-				<box size="0.30 0.10 0.07"/>
+				<box size="0.4172 0.116 0.03035"/>
 			</geometry>
 		</collision>
 		<inertial>
-			<mass value="2"/>
-			<inertia ixx="0.13" ixy="0.0" ixz="0.0" iyy="0.21" iyz="0.0" izz="0.13"/>
+			<mass value="0.500"/>
+			<inertia ixx="0.00093" ixy="0.0" ixz="0.0" iyy="0.00458" iyz="0.0" izz="0.00540"/>
 		</inertial>
 	</link>
@@ -53,5 +53,5 @@
 					<origin xyz="0 0 0" rpy="0 0 0" />
 					<geometry>
-						<box size="0.03 0.05 0.03"/>
+						<box size="0.060 0.035 0.078"/>
 					</geometry>
 					<material name="red"/>
@@ -60,10 +60,10 @@
 					<origin xyz="0 0 0" rpy="0 0 0" />
 					<geometry>
-						<box size="0.03 0.05 0.03"/>
-					</geometry>
-				</collision>
-				<inertial>
-					<mass value="0.1"/>
-					<inertia ixx="0.01" ixy="0.0" ixz="0.0" iyy="0.01" iyz="0.0" izz="0.01"/>
+						<box size="0.060 0.035 0.078"/>
+					</geometry>
+				</collision>
+				<inertial>
+					<mass value="0.332"/>
+					<inertia ixx="0.00109" ixy="0.0" ixz="-0.00004" iyy="0.00146" iyz="-0.00039" izz="0.00066"/>
 				</inertial>
 			</link>
@@ -102,19 +102,19 @@
 			<link name="link_${long}_${lat}_upperleg">
 				<visual>
-					<origin xyz="-0.075 0 0" rpy="0 0 0" />
-					<geometry>
-						<box size="${upperleg_length+0.03} 0.03 0.03"/>
+					<origin xyz="-0.07 0 0" rpy="0 0 0" />
+					<geometry>
+						<box size="${upperleg_length+0.03} 0.0365 0.026"/>
 					</geometry>
 					<material name="blue"/>
 				</visual>
 				<collision>
-					<origin xyz="-0.075 0 0" rpy="0 0 0" />
-					<geometry>
-						<box size="${upperleg_length+0.03}  0.03 0.03"/>
-					</geometry>
-				</collision>
-				<inertial>
-					<mass value="0.1"/>
-					<inertia ixx="0.1" ixy="0.0" ixz="0.0" iyy="0.1" iyz="0.0" izz="0.1"/>
+					<origin xyz="-0.07 0 0" rpy="0 0 0" />
+					<geometry>
+						<box size="${upperleg_length+0.03}  0.0365 0.026"/>
+					</geometry>
+				</collision>
+				<inertial>
+					<mass value="0.32114"/>
+					<inertia ixx="0.00014" ixy="0.00001" ixz="0.00002" iyy="0.00207" iyz="0.0" izz="0.00215"/>
 				</inertial>
 			</link>
@@ -149,5 +149,5 @@
 					<origin xyz="0.075 0 0" rpy="0 0 0" />
 					<geometry>
-						<box size="${lowerleg_length+0.03} 0.03 0.03"/>
+						<box size="${lowerleg_length+0.03} 0.02 0.03"/>
 					</geometry>
 					<material name="blue"/>
@@ -156,10 +156,10 @@
 					<origin xyz="0.075 0 0" rpy="0 0 0" />
 					<geometry>
-						<box size="${lowerleg_length+0.03} 0.03 0.03"/>
-					</geometry>
-				</collision>
-				<inertial>
-					<mass value="0.1"/>
-					<inertia ixx="0.1" ixy="0.0" ixz="0.0" iyy="0.1" iyz="0.0" izz="0.1"/>
+						<box size="${lowerleg_length+0.03} 0.02 0.03"/>
+					</geometry>
+				</collision>
+				<inertial>
+					<mass value="0.20407"/>
+					<inertia ixx="0.00005" ixy="0.00008" ixz="0.0" iyy="0.00121" iyz="0.0" izz="0.00123"/>
 				</inertial>
 			</link>
@@ -167,5 +167,5 @@
 				<parent link="link_${long}_${lat}_upperleg"/>
 				<child link="link_${long}_${lat}_lowerleg"/>
-				<origin xyz="-0.15 0 0" rpy="0 1.5708 0" />
+				<origin xyz="-0.15 0 -0.0156" rpy="0 1.5708 0" />
 				<axis xyz="0 1 0" />
 			</joint>
@@ -188,5 +188,5 @@
 					<origin xyz="0 0 0" rpy="0 0 0" />
 					<geometry>
-						<sphere radius = "0.03"/>
+						<sphere radius = "0.2"/>
 					</geometry>
 					<material name="green"/>
@@ -195,10 +195,10 @@
 					<origin xyz="0 0 0" rpy="0 0 0" />
 					<geometry>
-						<sphere radius = "0.03"/>
-					</geometry>
-				</collision>
-				<inertial>
-					<mass value="0.1"/>
-					<inertia ixx="0.1" ixy="0.0" ixz="0.0" iyy="0.1" iyz="0.0" izz="0.1"/>
+						<sphere radius = "0.2"/>
+					</geometry>
+				</collision>
+				<inertial>
+					<mass value="0.0"/>
+					<inertia ixx="0.0" ixy="0.0" ixz="0.0" iyy="0.0" iyz="0.0" izz="0.0"/>
 				</inertial>
 			</link>

Commit message: fixed error in urdf file

File: ros_packages/qd_simulation/robot_description/quadrus.xacro (robot description, xacro)
@@ -188,5 +188,5 @@
 					<origin xyz="0 0 0" rpy="0 0 0" />
 					<geometry>
-						<sphere radius = "0.2"/>
+						<sphere radius = "0.02"/>
 					</geometry>
 					<material name="green"/>
@@ -195,5 +195,5 @@
 					<origin xyz="0 0 0" rpy="0 0 0" />
 					<geometry>
-						<sphere radius = "0.2"/>
+						<sphere radius = "0.02"/>
 					</geometry>
 				</collision>

Commit message: Updated urdf file

File: ros_packages/qd_simulation/robot_description/quadrus.xacro (robot description, xacro)
@@ -3,7 +3,7 @@
 	<!-- Constants for robot dimensions, mass and inertia-->
 	<xacro:property name="PI" value="3.1415926535897931"/>
-	<xacro:property name="hip_offset" value="0.05755" />
-	<xacro:property name="upperleg_length" value="0.140" />
-	<xacro:property name="lowerleg_length" value="0.14833" />
+	<xacro:property name="hip_offset" value="0.05925" />
+	<xacro:property name="upperleg_length" value="0.13955" />
+	<xacro:property name="lowerleg_length" value="0.130" />
 	<xacro:property name="rear_hip_long_offset" value="-0.148" />
 	<xacro:property name="hip_long_center_dist" value="0.268" />
@@ -64,7 +64,7 @@
 				</collision>
 				<inertial>
-					<mass value="0.37017"/>
-					<origin xyz="0.00025 0.0063 0.04447"/>
-					<inertia ixx="0.00114" ixy="0.0" ixz="-0.00004" iyy="0.00074" iyz="-0.00021" izz="0.00064"/>
+					<mass value="0.1191"/>
+					<origin xyz="0.004136 0.002457 0.01974"/>
+					<inertia ixx="0.000176" ixy="-0.000004" ixz="-0.000017" iyy="0.000131" iyz="-0.000021" izz="0.000108"/>
 				</inertial>
 			</link>
@@ -116,7 +116,7 @@
 				</collision>
 				<inertial>
-					<mass value="0.35314"/>
-					<origin xyz="-0.06146 -0.00199 0.00083"/>
-					<inertia ixx="0.00015" ixy="-0.00003" ixz="0.00004" iyy="0.00074" iyz="0.0" izz="0.00083"/>
+					<mass value="0.13118"/>
+					<origin xyz="-0.041697 -0.007043 -0.000214"/>
+					<inertia ixx="0.000042" ixy="-0.000009" ixz="0.000011" iyy="0.000283" iyz="0.000002" izz="0.000310"/>
 				</inertial>
 			</link>
@@ -162,7 +162,7 @@
 				</collision>
 				<inertial>
-					<origin xyz=" 0.05439 0.00478 0"/>
-					<mass value="0.23649"/>
-					<inertia ixx="0.0" ixy="0.0" ixz="0.0" iyy="0.00052" iyz="0.0" izz="0.00054"/>
+					<mass value="0.10059"/>
+					<origin xyz=" 0.025048 -0.002594 0.000523"/>
+					<inertia ixx="0.000017" ixy="0.000001" ixz="0.000004" iyy="0.000149" iyz="0.0" izz="0.000158"/>
 				</inertial>
 			</link>
@@ -170,5 +170,5 @@
 				<parent link="link_${long}_${lat}_upperleg"/>
 				<child link="link_${long}_${lat}_lowerleg"/>
-				<origin xyz="-0.15 0 -0.0156" rpy="0 1.5708 0" />
+				<origin xyz="-0.15 0 -0.01886" rpy="0 1.5708 0" />
 				<axis xyz="0 1 0" />
 			</joint>
@@ -202,5 +202,5 @@
 				</collision>
 				<inertial>
-					<mass value="0.02"/>
+					<mass value="0.003"/>
 					<inertia ixx="0.0" ixy="0.0" ixz="0.0" iyy="0.0" iyz="0.0" izz="0.0"/>
 				</inertial>

Commit message: added collisions and gravity to gazebo

File: ros_packages/qd_simulation/robot_description/quadrus.xacro (robot description, xacro)
@@ -15,10 +15,10 @@
 	<xacro:include filename="$(find qd_simulation)/robot_description/quadrus.gazebo" />
 	<!-- Used for fixing robot to Gazebo 'base_link' -->
-	<link name="world"/>
+	<!-- link name="world"/>
 	<joint name="fixed" type="fixed">
 		<parent link="world"/>
 		<child link="base_link"/>
 		<origin xyz="0 0 1"/>
-	</joint>
+	</joint -->
 	<link name="base_link">
 		<visual>
@@ -108,4 +108,6 @@
 			<gazebo reference="link_${long}_${lat}_hip">
 				<material>Gazebo/Red</material>
+				<selfCollide>true</selfCollide>
+				<gravity>true</gravity>
 			</gazebo>
 		<!-- Upperleg -->
@@ -170,4 +172,6 @@
 			<gazebo reference="link_${long}_${lat}_upperleg">
 				<material>Gazebo/White</material>
+				<selfCollide>true</selfCollide>
+				<gravity>true</gravity>
 			</gazebo>
 		<!-- LowerLeg -->
@@ -227,4 +231,6 @@
 			<gazebo reference="link_${long}_${lat}_lowerleg">
 				<material>Gazebo/White</material>
+				<selfCollide>true</selfCollide>
+				<gravity>true</gravity>
 			</gazebo>
 		<!-- Paw -->
@@ -261,3 +267,4 @@
 	<xacro:quadrus_leg long="back" lat="left" id="3"/>
 	<xacro:quadrus_leg long="back" lat="right" id="4"/>
+	<selfCollide>true</selfCollide>
 </robot>

Commit message: added dummy link in urdf desc.

File: ros_packages/qd_simulation/robot_description/quadrus.xacro (robot description, xacro)
@@ -14,31 +14,36 @@
 	<!-- Import all Gazebo-customization elements, including Gazebo colors -->
 	<xacro:include filename="$(find qd_simulation)/robot_description/quadrus.gazebo" />
-	<!-- Used for fixing robot to Gazebo 'base_link' -->
-	<!-- link name="world"/>
-	<joint name="fixed" type="fixed">
-		<parent link="world"/>
-		<child link="base_link"/>
-		<origin xyz="0 0 1"/>
-	</joint -->
-	<link name="base_link">
-		<visual>
-			<origin xyz="0 0 0" rpy="0 0 0" />
-			<geometry>
-				<mesh filename="package://qd_simulation/robot_description/mesh/body.dae"/>
-			</geometry>
-			<material name="blue" />
-		</visual>
-		<collision>
-			<origin xyz="0 0 0" rpy="0 0 0" />
-			<geometry>
-				<box size="0.417 0.116 0.03"/>
-				<!-- mesh filename="package://qd_simulation/robot_description/mesh/body.dae"/-->
-			</geometry>
-		</collision>
-		<inertial>
-			<mass value="0.800"/>
-			<inertia ixx="0.00228" ixy="0.0" ixz="0.0" iyy="0.01125" iyz="0.0" izz="0.01326"/>
-		</inertial>
-	</link>
+	<!-- Used for fixing robot to Gazebo's base link -->
+	<link name="base_link"/>
+	<joint name="floating" type="fixed">
+		<parent link="base_link"/>
+		<child link="chassis"/>
+		<origin xyz="0 0 0"/>
+	</joint>
+	<!-- Chassis -->
+		<link name="chassis">
+			<visual>
+				<origin xyz="0 0 0" rpy="0 0 0" />
+				<geometry>
+					<mesh filename="package://qd_simulation/robot_description/mesh/body.dae"/>
+				</geometry>
+				<material name="blue" />
+			</visual>
+			<collision>
+				<origin xyz="0 0 0" rpy="0 0 0" />
+				<geometry>
+					<box size="0.417 0.116 0.03"/>
+					<!-- mesh filename="package://qd_simulation/robot_description/mesh/body.dae"/-->
+				</geometry>
+			</collision>
+			<inertial>
+				<mass value="0.800"/>
+				<inertia ixx="0.00228" ixy="0.0" ixz="0.0" iyy="0.01125" iyz="0.0" izz="0.01326"/>
+			</inertial>
+		</link>
+		<gazebo reference="chassis">
+			<material>Gazebo/Blue</material>
+			<gravity>true</gravity>
+		</gazebo>
 	<xacro:macro name="quadrus_leg" params="long lat id">
 		<!-- Hip -->
@@ -83,5 +88,5 @@
 			</link>
 			<joint name="${hip_joint_id}" type="continuous">
-				<parent link="base_link"/>
+				<parent link="chassis"/>
 				<child link="link_${long}_${lat}_hip"/>
 				<xacro:if value="${long == 'front' and lat == 'left'}">

Commit message: updated urdf file (body values)

File: ros_packages/qd_simulation/robot_description/quadrus.xacro (robot description, xacro)
@@ -7,7 +7,7 @@
 	<xacro:property name="upperleg_offset" value="0.01886" />
 	<xacro:property name="lowerleg_length" value="0.1296" />
-	<xacro:property name="rear_hip_long_offset" value="-0.148" />
-	<xacro:property name="hip_long_center_dist" value="0.268" />
-	<xacro:property name="hip_lat_center_dist" value="0.158" />
+	<xacro:property name="rear_hip_long_offset" value="-0.1486" />
+	<xacro:property name="hip_long_center_dist" value="0.2686" />
+	<xacro:property name="hip_lat_center_dist" value="0.178" />
 	<!-- Import Rviz colors -->
 	<xacro:include filename="$(find qd_simulation)/robot_description/materials.xacro" />
@@ -33,11 +33,12 @@
 				<origin xyz="0 0 0" rpy="0 0 0" />
 				<geometry>
-					<box size="0.417 0.116 0.03"/>
+					<box size="0.4172 0.136 0.03"/>
 					<!-- mesh filename="package://qd_simulation/robot_description/mesh/body.dae"/-->
 				</geometry>
 			</collision>
 			<inertial>
-				<mass value="0.800"/>
-				<inertia ixx="0.00228" ixy="0.0" ixz="0.0" iyy="0.01125" iyz="0.0" izz="0.01326"/>
+				<mass value="0.97859"/>
+				<origin xyz="-0.01428 0.00536 -0.00018"/>
+				<inertia ixx="0.00307" ixy="-0.00006" ixz="0.00006" iyy="0.01728" iyz="0.00003" izz="0.02001"/>
 			</inertial>
 		</link>
@@ -83,5 +84,5 @@
 				<inertial>
 					<mass value="0.1191"/>
-					<origin xyz="0.004136 0.002457 0.01974"/>
+					<origin xyz="0.00364 0.0025 0.01974"/>
 					<inertia ixx="0.000176" ixy="-0.000004" ixz="-0.000017" iyy="0.000131" iyz="-0.000021" izz="0.000108"/>
 				</inertial>
