Commit message: hw interface + launch files

File: ros_packages/qd_simulation/robot_description/quadrus.urdf (robot description, URDF)
Before this commit: robot quadrus, 18 links, 17 joints
Joints:
- removed joint joint_back_left_hip
- removed joint joint_back_left_lowerleg
- removed joint joint_back_left_upperleg
- removed joint joint_back_right_hip
- removed joint joint_back_right_lowerleg
- removed joint joint_back_right_upperleg
- removed joint joint_front_left_hip
- removed joint joint_front_left_lowerleg
- removed joint joint_front_left_upperleg
- removed joint joint_front_right_hip
- removed joint joint_front_right_lowerleg
- removed joint joint_front_right_upperleg
- added joint J1: type continuous, parent base_link, child link_front_left_hip, origin xyz=0.12 0.075 0 rpy=0 0 0, axis 1 0 0
- added joint J10: type continuous, parent base_link, child link_back_right_hip, origin xyz=-0.12 -0.075 0 rpy=0 0 0, axis 1 0 0
- added joint J11: type continuous, parent link_back_right_hip, child link_back_right_upperleg, origin xyz=0 -0.04 0 rpy=0 -0.7854 0, axis 0 1 0
- added joint J12: type continuous, parent link_back_right_upperleg, child link_back_right_lowerleg, origin xyz=-0.15 0 0 rpy=0 1.5708 0, axis 0 1 0
- added joint J2: type continuous, parent link_front_left_hip, child link_front_left_upperleg, origin xyz=0 0.04 0 rpy=0 -0.7854 0, axis 0 1 0
- added joint J3: type continuous, parent link_front_left_upperleg, child link_front_left_lowerleg, origin xyz=-0.15 0 0 rpy=0 1.5708 0, axis 0 1 0
- added joint J4: type continuous, parent base_link, child link_front_right_hip, origin xyz=0.12 -0.075 0 rpy=0 0 0, axis 1 0 0
- added joint J5: type continuous, parent link_front_right_hip, child link_front_right_upperleg, origin xyz=0 -0.04 0 rpy=0 -0.7854 0, axis 0 1 0
- added joint J6: type continuous, parent link_front_right_upperleg, child link_front_right_lowerleg, origin xyz=-0.15 0 0 rpy=0 1.5708 0, axis 0 1 0
- added joint J7: type continuous, parent base_link, child link_back_left_hip, origin xyz=-0.12 0.075 0 rpy=0 0 0, axis 1 0 0
- added joint J8: type continuous, parent link_back_left_hip, child link_back_left_upperleg, origin xyz=0 0.04 0 rpy=0 -0.7854 0, axis 0 1 0
- added joint J9: type continuous, parent link_back_left_upperleg, child link_back_left_lowerleg, origin xyz=-0.15 0 0 rpy=0 1.5708 0, axis 0 1 0

File: ros_packages/qd_simulation/robot_description/quadrus.xacro (robot description, xacro)
@@ -46,6 +46,7 @@
 		</inertial>
 	</link>
-	<xacro:macro name="quadrus_leg" params="long lat">
+	<xacro:macro name="quadrus_leg" params="long lat id">
 		<!-- Hip -->
+			<xacro:property name="hip_joint_id" value="J${(id-1)*3+1}"/>
 			<link name="link_${long}_${lat}_hip">
 				<visual>
@@ -67,5 +68,5 @@
 				</inertial>
 			</link>
-			<joint name="joint_${long}_${lat}_hip" type="continuous">
+			<joint name="${hip_joint_id}" type="continuous">
 				<parent link="base_link"/>
 				<child link="link_${long}_${lat}_hip"/>
@@ -86,5 +87,5 @@
 			<transmission name="transmission_${long}_${lat}_hip">
 				<type>transmission_interface/SimpleTransmission</type>
-				<joint name="joint_${long}_${lat}_hip">
+				<joint name="${hip_joint_id}">
 					<hardwareInterface>hardware_interface/EffortJointInterface</hardwareInterface>
 				</joint>
@@ -98,4 +99,5 @@
 			</gazebo>
 		<!-- Upperleg -->
+			<xacro:property name="upperleg_joint_id" value="J${(id-1)*3+2}"/>
 			<link name="link_${long}_${lat}_upperleg">
 				<visual>
@@ -117,5 +119,5 @@
 				</inertial>
 			</link>
-			<joint name="joint_${long}_${lat}_upperleg" type="continuous">
+			<joint name="${upperleg_joint_id}" type="continuous">
 				<parent link="link_${long}_${lat}_hip"/>
 				<child link="link_${long}_${lat}_upperleg"/>
@@ -130,5 +132,5 @@
 			<transmission name="transmission_${long}_${lat}_upperleg">
 				<type>transmission_interface/SimpleTransmission</type>
-				<joint name="joint_${long}_${lat}_upperleg">
+				<joint name="${upperleg_joint_id}">
 					<hardwareInterface>hardware_interface/EffortJointInterface</hardwareInterface>
 				</joint>
@@ -142,4 +144,5 @@
 			</gazebo>
 		<!-- LowerLeg -->
+			<xacro:property name="lowerleg_joint_id" value="J${(id-1)*3+3}"/>
 			<link name="link_${long}_${lat}_lowerleg">
 				<visual>
@@ -161,5 +164,5 @@
 				</inertial>
 			</link>
-			<joint name="joint_${long}_${lat}_lowerleg" type="continuous">
+			<joint name="${lowerleg_joint_id}" type="continuous">
 				<parent link="link_${long}_${lat}_upperleg"/>
 				<child link="link_${long}_${lat}_lowerleg"/>
@@ -169,5 +172,5 @@
 			<transmission name="transmission_${long}_${lat}_lowerleg">
 				<type>transmission_interface/SimpleTransmission</type>
-				<joint name="joint_${long}_${lat}_lowerleg">
+				<joint name="${lowerleg_joint_id}">
 					<hardwareInterface>hardware_interface/EffortJointInterface</hardwareInterface>
 				</joint>
@@ -209,4 +212,7 @@
 			</gazebo>
 	</xacro:macro>
-	<xacro:quadrus_leg long="back" lat="right"/>
+	<xacro:quadrus_leg long="front" lat="left" id="1"/>
+	<xacro:quadrus_leg long="front" lat="right" id="2"/>
+	<xacro:quadrus_leg long="back" lat="left" id="3"/>
+	<xacro:quadrus_leg long="back" lat="right" id="4"/>
 </robot>

Commit message: Updated joint limits in URDF for gazebo
Joints are now revolute instead of continuous. Also added gazebo_msgs dependency in CMake of qd_simulation

File: ros_packages/qd_simulation/robot_description/quadrus.urdf (robot description, URDF)
Before this commit: robot quadrus, 17 links, 16 joints
Links:
- added link chassis, mass 0.97859; collision box size=0.4172 0.136 0.03; visual mesh filename=package://qd_simulation/robot_description/mesh/body.dae
- link base_link: mass 0.800 -> None; geometry 
Joints:
- added joint floating: type fixed, parent base_link, child chassis, origin xyz=0 0 0
- joint J1: limit (none) -> lower=-0.401 upper=0.785 effort=30 velocity=10; origin xyz=0.12000000000000002 0.079 0 rpy=0 0 0 -> xyz=0.12 0.089 0 rpy=0 0 0; parent base_link -> chassis; type continuous -> revolute
- joint J10: limit (none) -> lower=-0.785 upper=0.401 effort=30 velocity=10; origin xyz=-0.148 -0.079 0 rpy=0 0 0 -> xyz=-0.1486 -0.089 0 rpy=0 0 0; parent base_link -> chassis; type continuous -> revolute
- joint J11: limit (none) -> lower=-1.5 upper=0.7 effort=1 velocity=1.0; type continuous -> revolute
- joint J12: limit (none) -> lower=-1.745 upper=1.396 effort=30 velocity=10; type continuous -> revolute
- joint J2: limit (none) -> lower=-1.5 upper=0.7 effort=30 velocity=10; type continuous -> revolute
- joint J3: limit (none) -> lower=-1.396 upper=1.745 effort=30 velocity=10; type continuous -> revolute
- joint J4: limit (none) -> lower=-0.785 upper=0.401 effort=30 velocity=10; origin xyz=0.12000000000000002 -0.079 0 rpy=0 0 0 -> xyz=0.12 -0.089 0 rpy=0 0 0; parent base_link -> chassis; type continuous -> revolute
- joint J5: limit (none) -> lower=-1.5 upper=0.7 effort=1 velocity=1.0; type continuous -> revolute
- joint J6: limit (none) -> lower=-1.745 upper=1.396 effort=30 velocity=10; type continuous -> revolute
- joint J7: limit (none) -> lower=-0.401 upper=0.785 effort=30 velocity=10; origin xyz=-0.148 0.079 0 rpy=0 0 0 -> xyz=-0.1486 0.089 0 rpy=0 0 0; parent base_link -> chassis; type continuous -> revolute
- joint J8: limit (none) -> lower=-1.5 upper=0.7 effort=30 velocity=10; type continuous -> revolute
- joint J9: limit (none) -> lower=-1.396 upper=1.745 effort=30 velocity=10; type continuous -> revolute

File: ros_packages/qd_simulation/robot_description/quadrus.xacro (robot description, xacro)
@@ -88,18 +88,22 @@
 				</inertial>
 			</link>
-			<joint name="${hip_joint_id}" type="continuous">
+			<joint name="${hip_joint_id}" type="revolute">
 				<parent link="chassis"/>
 				<child link="link_${long}_${lat}_hip"/>
 				<xacro:if value="${long == 'front' and lat == 'left'}">
 					<origin xyz="${rear_hip_long_offset+hip_long_center_dist} ${hip_lat_center_dist/2.0} 0" rpy="0 0 0" />
+					<limit effort="30" velocity="10" lower="-0.401" upper="0.785" />
 				</xacro:if>
 				<xacro:if value="${long == 'front' and lat == 'right'}">
 					<origin xyz="${rear_hip_long_offset+hip_long_center_dist} ${-hip_lat_center_dist/2.0} 0" rpy="0 0 0" />
+					<limit effort="30" velocity="10" lower="-0.785" upper="0.401" />
 				</xacro:if>
 				<xacro:if value="${long == 'back' and lat == 'left'}">
 					<origin xyz="${rear_hip_long_offset} ${hip_lat_center_dist/2.0} 0" rpy="0 0 0" />
+					<limit effort="30" velocity="10" lower="-0.401" upper="0.785" />
 				</xacro:if>
 				<xacro:if value="${long == 'back' and lat == 'right'}">
 					<origin xyz="${rear_hip_long_offset} ${-hip_lat_center_dist/2.0} 0" rpy="0 0 0" />
+					<limit effort="30" velocity="10" lower="-0.785" upper="0.401" />
 				</xacro:if>
 				<axis xyz="1 0 0" />
@@ -133,8 +137,8 @@
 						<origin xyz="0 0 0" rpy="0 0 0" />
 						<geometry>
-							<mesh filename="package://qd_simulation/robot_description/mesh/right_femur.dae"/>
-						</geometry>
-					</xacro:if>
-					<material name="blue"/>
+							<mesh filename="package://qd_simulation/robot_description/mesh/right_femur.dae" />
+						</geometry>
+					</xacro:if>
+					<material name="blue" />
 				</visual>
 				<collision>
@@ -160,12 +164,14 @@
 				</inertial>
 			</link>
-			<joint name="${upperleg_joint_id}" type="continuous">
+			<joint name="${upperleg_joint_id}" type="revolute">
 				<parent link="link_${long}_${lat}_hip"/>
 				<child link="link_${long}_${lat}_upperleg"/>
 				<xacro:if value="${lat == 'left'}">
 					<origin xyz="0 ${hip_offset} 0" rpy="0 0 0" />
+					<limit effort="30" velocity="10" lower="-1.5" upper="0.7" />
 				</xacro:if>
 				<xacro:if value="${lat == 'right'}">
 					<origin xyz="0 ${-hip_offset} 0" rpy="0 0 0" />
+					<limit effort="1" velocity="1.0" lower="-1.5" upper="0.7" />
 				</xacro:if>
 				<axis xyz="0 1 0" />
@@ -226,9 +232,15 @@
 				</inertial>
 			</link>
-			<joint name="${lowerleg_joint_id}" type="continuous">
+			<joint name="${lowerleg_joint_id}" type="revolute">
 				<parent link="link_${long}_${lat}_upperleg"/>
 				<child link="link_${long}_${lat}_lowerleg"/>
 				<origin xyz="${-upperleg_length} 0 ${-upperleg_offset}" rpy="0 1.5708 0" />
 				<axis xyz="0 1 0" />
+				<xacro:if value="${lat == 'right'}">
+					<limit effort="30" velocity="10" lower="-1.745" upper="1.396" />
+				</xacro:if>
+				<xacro:if value="${lat == 'left'}">
+					<limit effort="30" velocity="10" lower="-1.396" upper="1.745" />
+				</xacro:if>
 			</joint>
 			<transmission name="transmission_${long}_${lat}_lowerleg">
